Commit message: Fixed macro file for motoman

File: motoman_description/urdf/aprs_motoman.ros2_control.xacro (robot description, xacro)
@@ -1,7 +1,5 @@
 <?xml version="1.0"?>
 <robot xmlns:xacro="http://www.ros.org/wiki/xacro">
-  <xacro:macro name="aprs_motoman_ros2_control" params="
-    name
-    initial_positions">
+  <xacro:macro name="aprs_motoman_ros2_control" params="name">
     <ros2_control name="${name}" type="system">
       <hardware>
@@ -14,5 +12,4 @@
           </command_interface>
           <state_interface name="position">
-          <param name="initial_value">${initial_positions['joint_b']}</param>
           </state_interface>
           <state_interface name="velocity"/>
@@ -25,5 +22,4 @@
           </command_interface>
           <state_interface name="position">
-          <param name="initial_value">${initial_positions['joint_e']}</param>
           </state_interface>
           <state_interface name="velocity"/>
@@ -36,5 +32,4 @@
           </command_interface>
           <state_interface name="position">
-          <param name="initial_value">${initial_positions['joint_l']}</param>
           </state_interface>
           <state_interface name="velocity"/>
@@ -47,5 +42,4 @@
           </command_interface>
           <state_interface name="position">
-          <param name="initial_value">${initial_positions['joint_r']}</param>
           </state_interface>
           <state_interface name="velocity"/>
@@ -58,5 +52,4 @@
           </command_interface>
           <state_interface name="position">
-          <param name="initial_value">${initial_positions['joint_s']}</param>
           </state_interface>
           <state_interface name="velocity"/>
@@ -69,5 +62,4 @@
           </command_interface>
           <state_interface name="position">
-          <param name="initial_value">${initial_positions['joint_t']}</param>
           </state_interface>
           <state_interface name="velocity"/>
@@ -80,5 +72,4 @@
           </command_interface>
           <state_interface name="position">
-          <param name="initial_value">${initial_positions['joint_u']}</param>
           </state_interface>
           <state_interface name="velocity"/>

File: motoman_description/urdf/aprs_motoman_macro.xacro (robot description, xacro)
@@ -10,5 +10,4 @@
     <!-- Inclue gripper macro -->
     <!-- <xacro:include filename="$(find aprs_description)/urdf/vacuum_gripper/vacuum_grippper_macro.xacro"/> -->
-    <xacro:property name="initial_positions_file" default="$(find aprs_description)/config/motoman_initial_positions.yaml"/>
     <!-- Run motoman macro -->
     <xacro:motoman_sia20d
@@ -16,8 +15,5 @@
     </xacro:motoman_sia20d>
     <!-- Run motoman macro -->
-    <xacro:aprs_motoman_ros2_control
-      name="motoman"
-      initial_positions="${xacro.load_yaml(initial_positions_file)}">
-    </xacro:aprs_motoman_ros2_control>
+    <xacro:aprs_motoman_ros2_control name="motoman"/>
     <!-- Run gripper macro -->
     <!-- <xacro:vacuum_gripper

Commit message: Added motoman_moveit_config and updated joint names

File: motoman_description/urdf/aprs_motoman.ros2_control.xacro (robot description, xacro)
@@ -6,5 +6,5 @@
         <plugin>gz_ros2_control/GazeboSimSystem</plugin>
       </hardware>
-      <joint name="joint_b">
+      <joint name="joint_5">
           <command_interface name="position">
           <param name="min">{-2*pi}</param>
@@ -16,5 +16,5 @@
           <state_interface name="effort"/>
       </joint>
-      <joint name="joint_e">
+      <joint name="joint_7">
           <command_interface name="position">
           <param name="min">{-2*pi}</param>
@@ -26,5 +26,5 @@
           <state_interface name="effort"/>
       </joint>
-      <joint name="joint_l">
+      <joint name="joint_2">
           <command_interface name="position">
           <param name="min">{-pi}</param>
@@ -36,5 +36,5 @@
           <state_interface name="effort"/>
       </joint>
-      <joint name="joint_r">
+      <joint name="joint_4">
           <command_interface name="position">
           <param name="min">{-2*pi}</param>
@@ -46,5 +46,5 @@
           <state_interface name="effort"/>
       </joint>
-      <joint name="joint_s">
+      <joint name="joint_1">
           <command_interface name="position">
           <param name="min">{-2*pi}</param>
@@ -56,5 +56,5 @@
           <state_interface name="effort"/>
       </joint>
-      <joint name="joint_t">
+      <joint name="joint_6">
           <command_interface name="position">
           <param name="min">{-2*pi}</param>
@@ -66,5 +66,5 @@
           <state_interface name="effort"/>
       </joint>
-      <joint name="joint_u">
+      <joint name="joint_3">
           <command_interface name="position">
           <param name="min">{-2*pi}</param>

File: motoman_description/urdf/motoman_common.xacro (robot description, xacro)
@@ -52,23 +52,23 @@
 		<!-- <safety_controller soft_upper="0" soft_lower="0" k_position="0" k_velocity="0"/> -->
 	</xacro:macro>
-	<xacro:macro name="origin_joint_s">
+	<xacro:macro name="origin_joint_1">
         <origin xyz="0 0 0.112" rpy="1.5708 0 0" />
 	</xacro:macro>
-	<xacro:macro name="origin_joint_l">
+	<xacro:macro name="origin_joint_2">
         <origin xyz="0 0.298 0" rpy="0 0 0" />
 	</xacro:macro>
-	<xacro:macro name="origin_joint_e">
+	<xacro:macro name="origin_joint_7">
         <origin xyz="0 0.247135547651375 0" rpy="0 0 0" />
 	</xacro:macro>
-	<xacro:macro name="origin_joint_u">
+	<xacro:macro name="origin_joint_3">
         <origin xyz="0 0.242864452348634 0" rpy="0 0 0" />
 	</xacro:macro>
-	<xacro:macro name="origin_joint_r">
+	<xacro:macro name="origin_joint_4">
         <origin xyz="0 0.23899999999989 0" rpy="0 0 0" />
 	</xacro:macro>
-	<xacro:macro name="origin_joint_b">
+	<xacro:macro name="origin_joint_5">
         <origin xyz="0 0.181 0" rpy="0 0 0" />
 	</xacro:macro>
-	<xacro:macro name="origin_joint_t">
+	<xacro:macro name="origin_joint_6">
         <origin xyz="0 0.164069662461231 0.0015" rpy="0 0 0" />
 	</xacro:macro>

File: motoman_description/urdf/motoman_sia20_macro.xacro (robot description, xacro)
@@ -43,6 +43,6 @@
 			<child link = "motoman_base_link"/>
       	</joint>
-		<joint name="joint_s" type="revolute">
-			<xacro:origin_joint_s/>
+		<joint name="joint_1" type="revolute">
+			<xacro:origin_joint_1/>
 			<parent link="motoman_base_link"/>
 			<child  link="link_s"/>
@@ -67,7 +67,7 @@
 			</collision>
 		</link>
-		<!-- joint_l (link_s | joint_l) -->
-		<joint name="joint_l" type="revolute">
-			<xacro:origin_joint_l/>
+		<!-- joint_2 (link_s | joint_2) -->
+		<joint name="joint_2" type="revolute">
+			<xacro:origin_joint_2/>
 			<parent link="link_s"/>
 			<child  link="link_l"/>
@@ -92,7 +92,7 @@
 			</collision>
 		</link>
-		<!-- joint_e (link_l | joint_e) -->
-		<joint name="joint_e" type="revolute">
-			<xacro:origin_joint_e/>
+		<!-- joint_7 (link_l | joint_7) -->
+		<joint name="joint_7" type="revolute">
+			<xacro:origin_joint_7/>
 			<parent link="link_l"/>
 			<child  link="link_e"/>
@@ -117,7 +117,7 @@
 			</collision>
 		</link>
-		<!-- joint_u (link_e | joint_u) -->
-		<joint name="joint_u" type="revolute">
-			<xacro:origin_joint_u/>
+		<!-- joint_3 (link_e | joint_3) -->
+		<joint name="joint_3" type="revolute">
+			<xacro:origin_joint_3/>
 			<parent link="link_e"/>
 			<child  link="link_u"/>
@@ -142,7 +142,7 @@
 			</collision>
 		</link>
-		<!-- joint_r (link_u | joint_r) -->
-		<joint name="joint_r" type="revolute">
-			<xacro:origin_joint_r/>
+		<!-- joint_4 (link_u | joint_4) -->
+		<joint name="joint_4" type="revolute">
+			<xacro:origin_joint_4/>
 			<parent link="link_u"/>
 			<child  link="link_r"/>
@@ -167,7 +167,7 @@
 			</collision>
 		</link>
-		<!-- joint_b (link_r | joint_b) -->
-		<joint name="joint_b" type="revolute">
-			<xacro:origin_joint_b/>
+		<!-- joint_5 (link_r | joint_5) -->
+		<joint name="joint_5" type="revolute">
+			<xacro:origin_joint_5/>
 			<parent link="link_r"/>
 			<child  link="link_b"/>
@@ -192,7 +192,7 @@
 			</collision>
 		</link>
-		<!-- joint_t (link_b | joint_t) -->
-		<joint name="joint_t" type="revolute">
-			<xacro:origin_joint_t/>
+		<!-- joint_6 (link_b | joint_6) -->
+		<joint name="joint_6" type="revolute">
+			<xacro:origin_joint_6/>
 			<parent link="link_b"/>
 			<child  link="link_t"/>
