Commit message: Move group starts correctly

File: motoman_description/urdf/motoman.ros2_control.xacro (robot description, xacro)
@@ -1,10 +1,10 @@
 <?xml version="1.0"?>
 <robot xmlns:xacro="http://www.ros.org/wiki/xacro">
-  <xacro:macro name="aprs_motoman_ros2_control" params="name">
+  <xacro:macro name="motoman_ros2_control" params="name">
     <ros2_control name="${name}" type="system">
       <hardware>
         <plugin>gz_ros2_control/GazeboSimSystem</plugin>
       </hardware>
-      <joint name="joint_5">
+      <joint name="group_1/joint_5">
           <command_interface name="position">
           <param name="min">{-2*pi}</param>
@@ -16,5 +16,5 @@
           <state_interface name="effort"/>
       </joint>
-      <joint name="joint_7">
+      <joint name="group_1/joint_7">
           <command_interface name="position">
           <param name="min">{-2*pi}</param>
@@ -26,5 +26,5 @@
           <state_interface name="effort"/>
       </joint>
-      <joint name="joint_2">
+      <joint name="group_1/joint_2">
           <command_interface name="position">
           <param name="min">{-pi}</param>
@@ -36,5 +36,5 @@
           <state_interface name="effort"/>
       </joint>
-      <joint name="joint_4">
+      <joint name="group_1/joint_4">
           <command_interface name="position">
           <param name="min">{-2*pi}</param>
@@ -46,5 +46,5 @@
           <state_interface name="effort"/>
       </joint>
-      <joint name="joint_1">
+      <joint name="group_1/joint_1">
           <command_interface name="position">
           <param name="min">{-2*pi}</param>
@@ -56,5 +56,5 @@
           <state_interface name="effort"/>
       </joint>
-      <joint name="joint_6">
+      <joint name="group_1/joint_6">
           <command_interface name="position">
           <param name="min">{-2*pi}</param>
@@ -66,5 +66,5 @@
           <state_interface name="effort"/>
       </joint>
-      <joint name="joint_3">
+      <joint name="group_1/joint_3">
           <command_interface name="position">
           <param name="min">{-2*pi}</param>

File: motoman_description/urdf/motoman.urdf.xacro (robot description, xacro)
@@ -1,19 +1,15 @@
 <?xml version="1.0" ?>
-<robot xmlns:xacro="http://wiki.ros.org/xacro">
-  <xacro:macro name="aprs_motoman" params="
-    parent
-">
+<robot xmlns:xacro="http://wiki.ros.org/xacro" name="motoman">
     <!-- Inclue motoman robot macro -->
     <xacro:include filename="$(find motoman_description)/urdf/motoman_sia20_macro.xacro"/>
     <!-- Include ROS2 Control macro -->
-    <xacro:include filename="$(find motoman_description)/urdf/aprs_motoman.ros2_control.xacro"/>
+    <xacro:include filename="$(find motoman_description)/urdf/motoman.ros2_control.xacro"/>
     <!-- Inclue gripper macro -->
     <!-- <xacro:include filename="$(find aprs_description)/urdf/vacuum_gripper/vacuum_grippper_macro.xacro"/> -->
+    <link name="world"/>
     <!-- Run motoman macro -->
-    <xacro:motoman_sia20d
-        parent="${parent}">
-    </xacro:motoman_sia20d>
+    <xacro:motoman_sia20d parent="world"/>
     <!-- Run motoman macro -->
-    <xacro:aprs_motoman_ros2_control name="motoman"/>
+    <xacro:motoman_ros2_control name="motoman"/>
     <!-- Run gripper macro -->
     <!-- <xacro:vacuum_gripper
@@ -21,5 +17,4 @@
       prefix="motoman"
       > -->
-    </xacro:vacuum_gripper>
-  </xacro:macro>
+    <!-- </xacro:vacuum_gripper> -->
 </robot>

File: motoman_description/urdf/motoman_common.xacro (robot description, xacro)
@@ -8,5 +8,5 @@
 	<xacro:macro name="default_mesh" params="name">
 		<geometry>
-			<mesh filename="file://$(find aprs_description)/meshes/motoman/${name}.STL"/>
+			<mesh filename="file://$(find motoman_description)/meshes/${name}.STL"/>
 		</geometry>
 	</xacro:macro>
@@ -52,23 +52,23 @@
 		<!-- <safety_controller soft_upper="0" soft_lower="0" k_position="0" k_velocity="0"/> -->
 	</xacro:macro>
-	<xacro:macro name="origin_joint_1">
+	<xacro:macro name="origin_group_1_joint_1">
         <origin xyz="0 0 0.112" rpy="1.5708 0 0" />
 	</xacro:macro>
-	<xacro:macro name="origin_joint_2">
+	<xacro:macro name="origin_group_1_joint_2">
         <origin xyz="0 0.298 0" rpy="0 0 0" />
 	</xacro:macro>
-	<xacro:macro name="origin_joint_7">
+	<xacro:macro name="origin_group_1_joint_7">
         <origin xyz="0 0.247135547651375 0" rpy="0 0 0" />
 	</xacro:macro>
-	<xacro:macro name="origin_joint_3">
+	<xacro:macro name="origin_group_1_joint_3">
         <origin xyz="0 0.242864452348634 0" rpy="0 0 0" />
 	</xacro:macro>
-	<xacro:macro name="origin_joint_4">
+	<xacro:macro name="origin_group_1_joint_4">
         <origin xyz="0 0.23899999999989 0" rpy="0 0 0" />
 	</xacro:macro>
-	<xacro:macro name="origin_joint_5">
+	<xacro:macro name="origin_group_1_joint_5">
         <origin xyz="0 0.181 0" rpy="0 0 0" />
 	</xacro:macro>
-	<xacro:macro name="origin_joint_6">
+	<xacro:macro name="origin_group_1_joint_6">
         <origin xyz="0 0.164069662461231 0.0015" rpy="0 0 0" />
 	</xacro:macro>

File: motoman_description/urdf/motoman_sia20_macro.xacro (robot description, xacro)
@@ -2,5 +2,5 @@
 <robot name="motoman_sia20d" xmlns:xacro="http://www.ros.org/wiki/xacro">
 	<!-- include macro file-->
-	<xacro:include filename="$(find aprs_description)/urdf/motoman/motoman_common.xacro"/>
+	<xacro:include filename="$(find motoman_description)/urdf/motoman_common.xacro"/>
     <xacro:macro name="motoman_sia20d" params="parent">
 	<!-- motoman_base_link-->
@@ -43,6 +43,6 @@
 			<child link = "motoman_base_link"/>
       	</joint>
-		<joint name="joint_1" type="revolute">
-			<xacro:origin_joint_1/>
+		<joint name="group_1/joint_1" type="revolute">
+			<xacro:origin_group_1_joint_1/>
 			<parent link="motoman_base_link"/>
 			<child  link="link_s"/>
@@ -67,7 +67,7 @@
 			</collision>
 		</link>
-		<!-- joint_2 (link_s | joint_2) -->
-		<joint name="joint_2" type="revolute">
-			<xacro:origin_joint_2/>
+		<!-- group_1/joint_2 (link_s | group_1/joint_2) -->
+		<joint name="group_1/joint_2" type="revolute">
+			<xacro:origin_group_1_joint_2/>
 			<parent link="link_s"/>
 			<child  link="link_l"/>
@@ -92,7 +92,7 @@
 			</collision>
 		</link>
-		<!-- joint_7 (link_l | joint_7) -->
-		<joint name="joint_7" type="revolute">
-			<xacro:origin_joint_7/>
+		<!-- group_1/joint_7 (link_l | group_1/joint_7) -->
+		<joint name="group_1/joint_7" type="revolute">
+			<xacro:origin_group_1_joint_7/>
 			<parent link="link_l"/>
 			<child  link="link_e"/>
@@ -117,7 +117,7 @@
 			</collision>
 		</link>
-		<!-- joint_3 (link_e | joint_3) -->
-		<joint name="joint_3" type="revolute">
-			<xacro:origin_joint_3/>
+		<!-- group_1/joint_3 (link_e | group_1/joint_3) -->
+		<joint name="group_1/joint_3" type="revolute">
+			<xacro:origin_group_1_joint_3/>
 			<parent link="link_e"/>
 			<child  link="link_u"/>
@@ -142,7 +142,7 @@
 			</collision>
 		</link>
-		<!-- joint_4 (link_u | joint_4) -->
-		<joint name="joint_4" type="revolute">
-			<xacro:origin_joint_4/>
+		<!-- group_1/joint_4 (link_u | group_1/joint_4) -->
+		<joint name="group_1/joint_4" type="revolute">
+			<xacro:origin_group_1_joint_4/>
 			<parent link="link_u"/>
 			<child  link="link_r"/>
@@ -167,7 +167,7 @@
 			</collision>
 		</link>
-		<!-- joint_5 (link_r | joint_5) -->
-		<joint name="joint_5" type="revolute">
-			<xacro:origin_joint_5/>
+		<!-- group_1/joint_5 (link_r | group_1/joint_5) -->
+		<joint name="group_1/joint_5" type="revolute">
+			<xacro:origin_group_1_joint_5/>
 			<parent link="link_r"/>
 			<child  link="link_b"/>
@@ -192,7 +192,7 @@
 			</collision>
 		</link>
-		<!-- joint_6 (link_b | joint_6) -->
-		<joint name="joint_6" type="revolute">
-			<xacro:origin_joint_6/>
+		<!-- group_1/joint_6 (link_b | group_1/joint_6) -->
+		<joint name="group_1/joint_6" type="revolute">
+			<xacro:origin_group_1_joint_6/>
 			<parent link="link_b"/>
 			<child  link="link_t"/>

Commit message: Updates

File: motoman_description/urdf/motoman.ros2_control.xacro (robot description, xacro)
@@ -6,5 +6,5 @@
         <plugin>motoman_hardware/MotomanHardwareInterface</plugin>
       </hardware>
-      <joint name="group_1/joint_5">
+      <joint name="joint_s">
           <command_interface name="position">
           <param name="min">{-2*pi}</param>
@@ -14,5 +14,5 @@
           </state_interface>
       </joint>
-      <joint name="group_1/joint_7">
+      <joint name="joint_l">
           <command_interface name="position">
           <param name="min">{-2*pi}</param>
@@ -22,5 +22,5 @@
           </state_interface>
       </joint>
-      <joint name="group_1/joint_2">
+      <joint name="joint_e">
           <command_interface name="position">
           <param name="min">{-pi}</param>
@@ -30,5 +30,5 @@
           </state_interface>
       </joint>
-      <joint name="group_1/joint_4">
+      <joint name="joint_u">
           <command_interface name="position">
           <param name="min">{-2*pi}</param>
@@ -38,5 +38,5 @@
           </state_interface>
       </joint>
-      <joint name="group_1/joint_1">
+      <joint name="joint_r">
           <command_interface name="position">
           <param name="min">{-2*pi}</param>
@@ -46,5 +46,5 @@
           </state_interface>
       </joint>
-      <joint name="group_1/joint_6">
+      <joint name="joint_b">
           <command_interface name="position">
           <param name="min">{-2*pi}</param>
@@ -54,5 +54,5 @@
           </state_interface>
       </joint>
-      <joint name="group_1/joint_3">
+      <joint name="joint_t">
           <command_interface name="position">
           <param name="min">{-2*pi}</param>

File: motoman_description/urdf/motoman_common.xacro (robot description, xacro)
@@ -52,23 +52,23 @@
 		<!-- <safety_controller soft_upper="0" soft_lower="0" k_position="0" k_velocity="0"/> -->
 	</xacro:macro>
-	<xacro:macro name="origin_group_1_joint_1">
+	<xacro:macro name="origin_joint_r">
         <origin xyz="0 0 0.112" rpy="1.5708 0 0" />
 	</xacro:macro>
-	<xacro:macro name="origin_group_1_joint_2">
+	<xacro:macro name="origin_joint_e">
         <origin xyz="0 0.298 0" rpy="0 0 0" />
 	</xacro:macro>
-	<xacro:macro name="origin_group_1_joint_7">
+	<xacro:macro name="origin_joint_l">
         <origin xyz="0 0.247135547651375 0" rpy="0 0 0" />
 	</xacro:macro>
-	<xacro:macro name="origin_group_1_joint_3">
+	<xacro:macro name="origin_joint_t">
         <origin xyz="0 0.242864452348634 0" rpy="0 0 0" />
 	</xacro:macro>
-	<xacro:macro name="origin_group_1_joint_4">
+	<xacro:macro name="origin_joint_u">
         <origin xyz="0 0.23899999999989 0" rpy="0 0 0" />
 	</xacro:macro>
-	<xacro:macro name="origin_group_1_joint_5">
+	<xacro:macro name="origin_joint_s">
         <origin xyz="0 0.181 0" rpy="0 0 0" />
 	</xacro:macro>
-	<xacro:macro name="origin_group_1_joint_6">
+	<xacro:macro name="origin_joint_b">
         <origin xyz="0 0.164069662461231 0.0015" rpy="0 0 0" />
 	</xacro:macro>

File: motoman_description/urdf/motoman_sia20_macro.xacro (robot description, xacro)
@@ -43,6 +43,6 @@
 			<child link = "motoman_base_link"/>
       	</joint>
-		<joint name="group_1/joint_1" type="revolute">
-			<xacro:origin_group_1_joint_1/>
+		<joint name="joint_r" type="revolute">
+			<xacro:origin_joint_r/>
 			<parent link="motoman_base_link"/>
 			<child  link="link_s"/>
@@ -67,7 +67,7 @@
 			</collision>
 		</link>
-		<!-- group_1/joint_2 (link_s | group_1/joint_2) -->
-		<joint name="group_1/joint_2" type="revolute">
-			<xacro:origin_group_1_joint_2/>
+		<!-- joint_e (link_s | joint_e) -->
+		<joint name="joint_e" type="revolute">
+			<xacro:origin_joint_e/>
 			<parent link="link_s"/>
 			<child  link="link_l"/>
@@ -92,7 +92,7 @@
 			</collision>
 		</link>
-		<!-- group_1/joint_7 (link_l | group_1/joint_7) -->
-		<joint name="group_1/joint_7" type="revolute">
-			<xacro:origin_group_1_joint_7/>
+		<!-- joint_l (link_l | joint_l) -->
+		<joint name="joint_l" type="revolute">
+			<xacro:origin_joint_l/>
 			<parent link="link_l"/>
 			<child  link="link_e"/>
@@ -117,7 +117,7 @@
 			</collision>
 		</link>
-		<!-- group_1/joint_3 (link_e | group_1/joint_3) -->
-		<joint name="group_1/joint_3" type="revolute">
-			<xacro:origin_group_1_joint_3/>
+		<!-- joint_t (link_e | joint_t) -->
+		<joint name="joint_t" type="revolute">
+			<xacro:origin_joint_t/>
 			<parent link="link_e"/>
 			<child  link="link_u"/>
@@ -142,7 +142,7 @@
 			</collision>
 		</link>
-		<!-- group_1/joint_4 (link_u | group_1/joint_4) -->
-		<joint name="group_1/joint_4" type="revolute">
-			<xacro:origin_group_1_joint_4/>
+		<!-- joint_u (link_u | joint_u) -->
+		<joint name="joint_u" type="revolute">
+			<xacro:origin_joint_u/>
 			<parent link="link_u"/>
 			<child  link="link_r"/>
@@ -167,7 +167,7 @@
 			</collision>
 		</link>
-		<!-- group_1/joint_5 (link_r | group_1/joint_5) -->
-		<joint name="group_1/joint_5" type="revolute">
-			<xacro:origin_group_1_joint_5/>
+		<!-- joint_s (link_r | joint_s) -->
+		<joint name="joint_s" type="revolute">
+			<xacro:origin_joint_s/>
 			<parent link="link_r"/>
 			<child  link="link_b"/>
@@ -192,7 +192,7 @@
 			</collision>
 		</link>
-		<!-- group_1/joint_6 (link_b | group_1/joint_6) -->
-		<joint name="group_1/joint_6" type="revolute">
-			<xacro:origin_group_1_joint_6/>
+		<!-- joint_b (link_b | joint_b) -->
+		<joint name="joint_b" type="revolute">
+			<xacro:origin_joint_b/>
 			<parent link="link_b"/>
 			<child  link="link_t"/>
